File: kicad/polytonic_greek_keyboard/driver.kicad_sch (KiCad schematic)
At the start: 2 parts, among them J1 USB_C_Receptacle, J5 Conn_01x11_Pin

Commit message: [UPDATE] anotation issues
Parts:
- renumbered J1 to J3, J5 to J4
Changed lines of the file:
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@@
 		(dnp no)
 		(fields_autoplaced yes)
-		(property "Reference" "J5"
+		(property "Reference" "J4"
 			(at 149.86 95.25 90)
 			(effects
@@
 			(project "polytonic_greek_keyboard"
 				(path "/cbe25a1b-6c02-43c2-9ff9-ba274c7cf6a2/8498b325-11fd-4b20-a704-75ec3d8987ef"
-					(reference "J5")
+					(reference "J4")
 					(unit 1)
 				)
@@
 		(dnp no)
 		(fields_autoplaced yes)
-		(property "Reference" "J1"
+		(property "Reference" "J3"
 			(at 25.4 19.05 0)
 			(effects
@@
 			(project "polytonic_greek_keyboard"
 				(path "/cbe25a1b-6c02-43c2-9ff9-ba274c7cf6a2/8498b325-11fd-4b20-a704-75ec3d8987ef"
-					(reference "J1")
+					(reference "J3")
 					(unit 1)
 				)
@@
 		)
 		(instances
-			(project "keyboard_driver"
+			(project "polytonic_greek_keyboard"
 				(path "/cbe25a1b-6c02-43c2-9ff9-ba274c7cf6a2/8498b325-11fd-4b20-a704-75ec3d8987ef"
 					(page "8")
@@
 		)
 		(instances
-			(project "keyboard_driver"
+			(project "polytonic_greek_keyboard"
 				(path "/cbe25a1b-6c02-43c2-9ff9-ba274c7cf6a2/8498b325-11fd-4b20-a704-75ec3d8987ef"
 					(page "7")
@@
 		)
 		(instances
-			(project "keyboard_driver"
+			(project "polytonic_greek_keyboard"
 				(path "/cbe25a1b-6c02-43c2-9ff9-ba274c7cf6a2/8498b325-11fd-4b20-a704-75ec3d8987ef"
 					(page "5")
@@
 		)
 		(instances
-			(project "keyboard_driver"
+			(project "polytonic_greek_keyboard"
 				(path "/cbe25a1b-6c02-43c2-9ff9-ba274c7cf6a2/8498b325-11fd-4b20-a704-75ec3d8987ef"
 					(page "6")
@@
 		)
 		(instances
-			(project "keyboard_driver"
+			(project "polytonic_greek_keyboard"
 				(path "/cbe25a1b-6c02-43c2-9ff9-ba274c7cf6a2/8498b325-11fd-4b20-a704-75ec3d8987ef"
 					(page "3")
@@
 		)
 		(instances
-			(project "keyboard_driver"
+			(project "polytonic_greek_keyboard"
 				(path "/cbe25a1b-6c02-43c2-9ff9-ba274c7cf6a2/8498b325-11fd-4b20-a704-75ec3d8987ef"
 					(page "9")

Commit message: [UPDATE] the final merged version of the schematic before splitting into two separate kicad projects
Other:
- note added: "3.3V"
- note added: "5V"
- note added: "GND"
- note added: "LED_DIN"
- note added: "MCP1_INTA"
- note added: "MCP1_INTB"
- note added: "MCP2_INTA"
- note added: "MCP2_INTB"
- note added: "RESET"
- note added: "SCK"
- note added: "SDA"
- company: (none) -> Henry's Software House
- title: (none) -> Driver logic
Changed lines of the file:
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@@
 	(generator_version "9.0")
 	(paper "A4")
+	(title_block
+		(title "Driver logic")
+		(date "2026-02-10")
+		(rev "1 - do not edit connector pin layout.")
+		(company "Henry's Software House")
+		(comment 1 "The logic required to drive the keyboard.")
+		(comment 2 "Logic based on an ESP32-S2-wroover")
+	)
+	(text "RESET"
+		(exclude_from_sim no)
+		(at 145.034 96.266 90)
+		(effects
+			(font
+				(size 1.27 1.27)
+			)
+		)
+	)
+	(text "LED_DIN"
+		(exclude_from_sim no)
+		(at 157.734 97.028 90)
+		(effects
+			(font
+				(size 1.27 1.27)
+			)
+		)
+	)
+	(text "GND"
+		(exclude_from_sim no)
+		(at 137.16 95.758 90)
+		(effects
+			(font
+				(size 1.27 1.27)
+			)
+		)
+	)
+	(text "MCP1_INTA"
+		(exclude_from_sim no)
+		(at 147.574 98.552 90)
+		(effects
+			(font
+				(size 1.27 1.27)
+			)
+		)
+	)
+	(text "MCP2_INTB"
+		(exclude_from_sim no)
+		(at 155.194 98.298 90)
+		(effects
+			(font
+				(size 1.27 1.27)
+			)
+		)
+	)
+	(text "5V"
+		(exclude_from_sim no)
+		(at 139.7 95.25 90)
+		(effects
+			(font
+				(size 1.27 1.27)
+			)
+		)
+	)
+	(text "MCP1_INTB"
+		(exclude_from_sim no)
+		(at 150.114 98.552 90)
+		(effects
+			(font
+				(size 1.27 1.27)
+			)
+		)
+	)
+	(text "MCP2_INTA"
+		(exclude_from_sim no)
+		(at 152.654 98.298 90)
+		(effects
+			(font
+				(size 1.27 1.27)
+			)
+		)
+	)
+	(text "3.3V"
+		(exclude_from_sim no)
+		(at 142.494 96.012 90)
+		(effects
+			(font
+				(size 1.27 1.27)
+			)
+		)
+	)
+	(text "SDA"
+		(exclude_from_sim no)
+		(at 160.274 94.996 90)
+		(effects
+			(font
+				(size 1.27 1.27)
+			)
+		)
+	)
+	(text "SCK"
+		(exclude_from_sim no)
+		(at 162.814 94.996 90)
+		(effects
+			(font
+				(size 1.27 1.27)
+			)
+		)
+	)
 	(junction
 		(at 118.11 36.83)
@@
 		(on_board yes)
 		(dnp no)
-		(fields_autoplaced yes)
 		(property "Reference" "J4"
-			(at 149.86 95.25 90)
+			(at 171.45 89.408 90)
 			(effects
 				(font
@@
 		)
 		(property "Value" "Conn_01x11_Pin"
-			(at 149.86 97.79 90)
+			(at 171.45 91.948 90)
 			(effects
 				(font
