File: kicad/polytonic_greek_keyboard/keyboard_matrix.kicad_sch (KiCad schematic)
At the start: 3 parts, among them J4 Conn_01x11_Socket, U4 MCP23017_SP, U5 MCP23017_SP

Commit message: [UPDATE] anotation issues
Parts:
- renumbered J4 to J5
Changed lines of the file:
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@@
 		(dnp no)
 		(fields_autoplaced yes)
-		(property "Reference" "J4"
+		(property "Reference" "J5"
 			(at 92.71 13.97 90)
 			(effects
@@
 			(project "polytonic_greek_keyboard"
 				(path "/cbe25a1b-6c02-43c2-9ff9-ba274c7cf6a2/dc7dc8d0-3fc1-4401-9905-7f0a56042fcf"
-					(reference "J4")
+					(reference "J5")
 					(unit 1)
 				)
@@
 		)
 		(instances
-			(project "keyboard_driver"
+			(project "polytonic_greek_keyboard"
 				(path "/cbe25a1b-6c02-43c2-9ff9-ba274c7cf6a2/dc7dc8d0-3fc1-4401-9905-7f0a56042fcf"
 					(page "2")

Commit message: [UPDATE] the final merged version of the schematic before splitting into two separate kicad projects
Other:
- note added: "3.3V"
- note added: "5V"
- note added: "GND"
- note added: "LED_DIN"
- note added: "MCP1_INTA"
- note added: "MCP1_INTB"
- note added: "MCP2_INTA"
- note added: "MCP2_INTB"
- note added: "RESET"
- note added: "SCK"
- note added: "SDA"
- company: (none) -> Henry's Software House
- title: (none) -> Keyboard Matrix
- moved on the sheet: J5, U4, U5
