File: kicad/polytonic_greek_keyboard/navigation_keys.kicad_sch (KiCad schematic)
At the start: 0 parts

Commit message: [UPDATE] the final merged version of the schematic before splitting into two separate kicad projects
Other:
- company: (none) -> Henry's Software House
Changed lines of the file:
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@@
 	(generator_version "9.0")
 	(paper "A4")
+	(title_block
+		(rev "1 - do not edit connector pin layout.")
+		(company "Henry's Software House")
+	)
 	(wire
 		(pts
